File: Hardware/SparkFun_TensorFlow_Ambiq_Apollo3.brd (EAGLE design)
At the start: 40 x 40 mm, 132 parts, among them J5 CORTEX_DEBUG_PTH, J6 CAMERA-0V7670, M1 MEMS_MIC, M2 MEMS_MIC, U1 AMBIQ-APOLLO3KBR, U2 LIS2DH12, U3 1.8V, U4 LMV358, Y1 32MHz, Y2 32.768kHz

Commit message: Adding production ID's to all part numbers.
Parts:
- J6: value CAMERA-0V7670 -> CAMERA-OV7670
Changed lines of the file:
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@@
 <layer number="23" name="tOrigins" color="15" fill="1" visible="yes" active="yes"/>
 <layer number="24" name="bOrigins" color="15" fill="1" visible="yes" active="yes"/>
-<layer number="25" name="tNames" color="7" fill="1" visible="yes" active="yes"/>
-<layer number="26" name="bNames" color="7" fill="1" visible="yes" active="yes"/>
-<layer number="27" name="tValues" color="7" fill="1" visible="yes" active="yes"/>
-<layer number="28" name="bValues" color="7" fill="1" visible="yes" active="yes"/>
-<layer number="29" name="tStop" color="7" fill="3" visible="yes" active="yes"/>
-<layer number="30" name="bStop" color="7" fill="6" visible="yes" active="yes"/>
-<layer number="31" name="tCream" color="7" fill="4" visible="yes" active="yes"/>
-<layer number="32" name="bCream" color="7" fill="5" visible="yes" active="yes"/>
-<layer number="33" name="tFinish" color="6" fill="3" visible="yes" active="yes"/>
-<layer number="34" name="bFinish" color="6" fill="6" visible="yes" active="yes"/>
-<layer number="35" name="tGlue" color="7" fill="4" visible="yes" active="yes"/>
-<layer number="36" name="bGlue" color="7" fill="5" visible="yes" active="yes"/>
-<layer number="37" name="tTest" color="7" fill="1" visible="yes" active="yes"/>
-<layer number="38" name="bTest" color="7" fill="1" visible="yes" active="yes"/>
-<layer number="39" name="tKeepout" color="4" fill="11" visible="yes" active="yes"/>
-<layer number="40" name="bKeepout" color="1" fill="11" visible="yes" active="yes"/>
-<layer number="41" name="tRestrict" color="4" fill="10" visible="yes" active="yes"/>
-<layer number="42" name="bRestrict" color="1" fill="10" visible="yes" active="yes"/>
-<layer number="43" name="vRestrict" color="2" fill="10" visible="yes" active="yes"/>
-<layer number="44" name="Drills" color="7" fill="1" visible="yes" active="yes"/>
+<layer number="25" name="tNames" color="7" fill="1" visible="no" active="yes"/>
+<layer number="26" name="bNames" color="7" fill="1" visible="no" active="yes"/>
+<layer number="27" name="tValues" color="7" fill="1" visible="no" active="yes"/>
+<layer number="28" name="bValues" color="7" fill="1" visible="no" active="yes"/>
+<layer number="29" name="tStop" color="7" fill="3" visible="no" active="yes"/>
+<layer number="30" name="bStop" color="7" fill="6" visible="no" active="yes"/>
+<layer number="31" name="tCream" color="7" fill="4" visible="no" active="yes"/>
+<layer number="32" name="bCream" color="7" fill="5" visible="no" active="yes"/>
+<layer number="33" name="tFinish" color="6" fill="3" visible="no" active="yes"/>
+<layer number="34" name="bFinish" color="6" fill="6" visible="no" active="yes"/>
+<layer number="35" name="tGlue" color="7" fill="4" visible="no" active="yes"/>
+<layer number="36" name="bGlue" color="7" fill="5" visible="no" active="yes"/>
+<layer number="37" name="tTest" color="7" fill="1" visible="no" active="yes"/>
+<layer number="38" name="bTest" color="7" fill="1" visible="no" active="yes"/>
+<layer number="39" name="tKeepout" color="4" fill="11" visible="no" active="yes"/>
+<layer number="40" name="bKeepout" color="1" fill="11" visible="no" active="yes"/>
+<layer number="41" name="tRestrict" color="4" fill="10" visible="no" active="yes"/>
+<layer number="42" name="bRestrict" color="1" fill="10" visible="no" active="yes"/>
+<layer number="43" name="vRestrict" color="2" fill="10" visible="no" active="yes"/>
+<layer number="44" name="Drills" color="7" fill="1" visible="no" active="yes"/>
 <layer number="45" name="Holes" color="7" fill="1" visible="yes" active="yes"/>
-<layer number="46" name="Milling" color="3" fill="1" visible="yes" active="yes"/>
-<layer number="47" name="Measures" color="7" fill="1" visible="yes" active="yes"/>
-<layer number="48" name="Document" color="7" fill="1" visible="yes" active="yes"/>
-<layer number="49" name="Reference" color="7" fill="1" visible="yes" active="yes"/>
-<layer number="50" name="dxf" color="7" fill="1" visible="yes" active="yes"/>
+<layer number="46" name="Milling" color="3" fill="1" visible="no" active="yes"/>
+<layer number="47" name="Measures" color="7" fill="1" visible="no" active="yes"/>
+<layer number="48" name="Document" color="7" fill="1" visible="no" active="yes"/>
+<layer number="49" name="Reference" color="7" fill="1" visible="no" active="yes"/>
+<layer number="50" name="dxf" color="7" fill="1" visible="no" active="yes"/>
 <layer number="51" name="tDocu" color="6" fill="1" visible="yes" active="yes"/>
-<layer number="52" name="bDocu" color="7" fill="1" visible="yes" active="yes"/>
+<layer number="52" name="bDocu" color="7" fill="1" visible="no" active="yes"/>
 <layer number="91" name="Nets" color="2" fill="1" visible="no" active="no"/>
 <layer number="92" name="Busses" color="1" fill="1" visible="no" active="no"/>
@@
 <layer number="95" name="Names" color="7" fill="1" visible="no" active="no"/>
 <layer number="96" name="Values" color="7" fill="1" visible="no" active="no"/>
-<layer number="2" name="Route2" color="22" fill="3" visible="yes" active="yes"/>
-<layer number="15" name="Route15" color="14" fill="6" visible="yes" active="yes"/>
+<layer number="2" name="Route2" color="22" fill="3" visible="no" active="yes"/>
+<layer number="15" name="Route15" color="14" fill="6" visible="no" active="yes"/>
 <layer number="53" name="tGND_GNDA" color="7" fill="9" visible="no" active="no"/>
 <layer number="54" name="bGND_GNDA" color="1" fill="9" visible="no" active="no"/>
@@
 <element name="A1" library="ambiq" package="ANT-2.4GHZ-3.2X1.6X1.2MM" value="2.4GHZ-3.2X1.6MM" x="38.128" y="16.3" smashed="yes" rot="R270">
 <attribute name="DIGIKEY" value="535-14095-2-ND" x="38.128" y="16.3" size="1.778" layer="27" font="vector" ratio="15" rot="R270" display="off"/>
+<attribute name="PROD_ID" value="ANT-14235" x="38.128" y="16.3" size="1.778" layer="27" rot="R270" display="off"/>
 </element>
 <element name="J5" library="SparkFun-Connectors" package="2X5-PTH-1.27MM" value="CORTEX_DEBUG_PTH" x="32" y="29" smashed="yes" rot="MR270">
@@
 <attribute name="VALUE" x="8.001" y="1.0922" size="0.6096" layer="27" font="vector" ratio="20" rot="R180" align="bottom-center"/>
 </element>
-<element name="J6" library="ambiq" package="FPC-24-AMPHENOL-SFV24R-1STE1HLF" value="CAMERA-0V7670" x="20" y="37" smashed="yes" rot="R180">
+<element name="J6" library="ambiq" package="FPC-24-AMPHENOL-SFV24R-1STE1HLF" value="CAMERA-OV7670" x="20" y="37" smashed="yes" rot="R180">
 <attribute name="DIGIKEY" value="609-4320-2-ND" x="20" y="37" size="1.778" layer="27" rot="R180" display="off"/>
 <attribute name="NAME" x="20" y="39.3368" size="0.6096" layer="25" font="vector" ratio="20" rot="R180" align="top-center"/>

Commit message: Change to 100x gain with 1M ohm resistors for mics
Parts:
- R20, R21: value 100k -> 1M
Changed lines of the file:
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@@
 <?xml version="1.0" encoding="utf-8"?>
 <!DOCTYPE eagle SYSTEM "eagle.dtd">
-<eagle version="9.2.2">
+<eagle version="9.1.3">
 <drawing>
 <settings>
@@
 <attribute name="VALUE" x="12.0842" y="32" size="0.6096" layer="27" font="vector" ratio="20" rot="R90" align="top-center"/>
 </element>
-<element name="R21" library="SparkFun-Resistors" package="0603" value="100k" x="10.75" y="29.6" smashed="yes">
+<element name="R21" library="SparkFun-Resistors" package="0603" value="1M" x="10.75" y="29.6" smashed="yes">
 <attribute name="NAME" x="10.75" y="30.362" size="0.6096" layer="25" font="vector" ratio="20" align="bottom-center"/>
-<attribute name="PROD_ID" value="RES-07828" x="10.75" y="29.6" size="1.778" layer="27" display="off"/>
-<attribute name="VALUE" x="10.75" y="29.0412" size="0.6096" layer="27" font="vector" ratio="20" align="top-center"/>
+<attribute name="PROD_ID" value="RES-07868" x="10.75" y="29.6" size="1.778" layer="27" display="off"/>
+<attribute name="VALUE" value="1M" x="10.75" y="29.0412" size="0.6096" layer="27" font="vector" ratio="20" align="top-center"/>
 </element>
 <element name="C24" library="SparkFun-Capacitors" package="0603" value="4.7uF" x="10" y="32" smashed="yes" rot="R270">
@@
 <attribute name="VALUE" x="10.437" y="6.542" size="0.6096" layer="27" font="vector" ratio="20" rot="R270" align="top-center"/>
 </element>
-<element name="R20" library="SparkFun-Resistors" package="0603" value="100k" x="12" y="8" smashed="yes" rot="R180">
+<element name="R20" library="SparkFun-Resistors" package="0603" value="1M" x="12" y="8" smashed="yes" rot="R180">
 <attribute name="NAME" x="12" y="7.238" size="0.6096" layer="25" font="vector" ratio="20" rot="R180" align="bottom-center"/>
-<attribute name="PROD_ID" value="RES-07828" x="12" y="8" size="1.778" layer="27" rot="R180" display="off"/>
-<attribute name="VALUE" x="12" y="8.635" size="0.6096" layer="27" font="vector" ratio="20" rot="R180" align="top-center"/>
+<attribute name="PROD_ID" value="RES-07868" x="12" y="8" size="1.778" layer="27" rot="R180" display="off"/>
+<attribute name="VALUE" value="1M" x="12" y="8.635" size="0.6096" layer="27" font="vector" ratio="20" rot="R180" align="top-center"/>
 </element>
 <element name="C26" library="SparkFun-Capacitors" package="0603" value="4.7uF" x="12" y="5" smashed="yes">

Commit message: Change Mic gain to 75x
This is Pete's requested final gain value
Parts:
- R20, R21: value 1M -> 750K
Changed lines of the file:
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@@
 <attribute name="VALUE" x="12.0842" y="32" size="0.6096" layer="27" font="vector" ratio="20" rot="R90" align="top-center"/>
 </element>
-<element name="R21" library="SparkFun-Resistors" package="0603" value="1M" x="10.75" y="29.6" smashed="yes">
+<element name="R21" library="SparkFun-Resistors" package="0603" value="750K" x="10.75" y="29.6" smashed="yes">
 <attribute name="NAME" x="10.75" y="30.362" size="0.6096" layer="25" font="vector" ratio="20" align="bottom-center"/>
-<attribute name="PROD_ID" value="RES-07868" x="10.75" y="29.6" size="1.778" layer="27" display="off"/>
-<attribute name="VALUE" value="1M" x="10.75" y="29.0412" size="0.6096" layer="27" font="vector" ratio="20" align="top-center"/>
+<attribute name="PROD_ID" value="RES-13768" x="10.75" y="29.6" size="1.778" layer="27" display="off"/>
+<attribute name="VALUE" value="750K" x="10.75" y="29.0412" size="0.6096" layer="27" font="vector" ratio="20" align="top-center"/>
 </element>
 <element name="C24" library="SparkFun-Capacitors" package="0603" value="4.7uF" x="10" y="32" smashed="yes" rot="R270">
@@
 <attribute name="VALUE" x="10.437" y="6.542" size="0.6096" layer="27" font="vector" ratio="20" rot="R270" align="top-center"/>
 </element>
-<element name="R20" library="SparkFun-Resistors" package="0603" value="1M" x="12" y="8" smashed="yes" rot="R180">
+<element name="R20" library="SparkFun-Resistors" package="0603" value="750K" x="12" y="8" smashed="yes" rot="R180">
 <attribute name="NAME" x="12" y="7.238" size="0.6096" layer="25" font="vector" ratio="20" rot="R180" align="bottom-center"/>
-<attribute name="PROD_ID" value="RES-07868" x="12" y="8" size="1.778" layer="27" rot="R180" display="off"/>
-<attribute name="VALUE" value="1M" x="12" y="8.635" size="0.6096" layer="27" font="vector" ratio="20" rot="R180" align="top-center"/>
+<attribute name="PROD_ID" value="RES-13768" x="12" y="8" size="1.778" layer="27" rot="R180" display="off"/>
+<attribute name="VALUE" value="750K" x="12" y="8.635" size="0.6096" layer="27" font="vector" ratio="20" rot="R180" align="top-center"/>
 </element>
 <element name="C26" library="SparkFun-Capacitors" package="0603" value="4.7uF" x="12" y="5" smashed="yes">
