File: Hardware/SparkFun_TensorFlow_Ambiq_Apollo3.brd (EAGLE design)
At the start: 40 x 40 mm, 100 parts, among them J5 CORTEX_DEBUG, J6 CAMERA-OV7670, U2 LIS2DH12, U3 1.8V, U5 ARTEMIS_MODULESMD, Y2 32.768kHz

Commit message: Update silk
Parts:
- removed U$24: (no value), buzzard_labels:EDGE0
- added U$15: (no value), buzzard_labels (11):EDGE_20
Changed lines of the file:
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@@
 <element name="U$20" library="buzzard_labels" package="CAMERA3" value="" x="28.448" y="38.354" smashed="yes"/>
 <element name="U$21" library="PoweredBy_TF#jpg" package="POWEREDBY_TF#JPG" value="" x="32.766" y="12.3" smashed="yes"/>
-<element name="U$24" library="buzzard_labels" package="EDGE0" value="" x="16.891" y="25.654" smashed="yes"/>
 <element name="U$1" library="buzzard_labels" package="MIC00" value="" x="5.9182" y="39.243" smashed="yes"/>
 <element name="TP1" library="SparkFun-Connectors" package="PAD.03X.05" value="" x="34.29" y="35.56" smashed="yes" rot="MR0"/>
@@
 <element name="U$26" library="buzzard_labels (14)" package="182" value="" x="16.9" y="-0.1" smashed="yes" rot="R90"/>
 <element name="U$31" library="buzzard_labels (14)" package="193" value="" x="15" y="-0.1" smashed="yes" rot="R90"/>
+<element name="U$15" library="buzzard_labels (11)" package="EDGE_20" value="" x="16.891" y="25.654" smashed="yes"/>
 </elements>
 <signals>
@@
 <contactref element="U5" pad="SWDCK"/>
 <via x="39" y="22" extent="1-16" drill="0.3048"/>
-<wire x1="39.6048" y1="26.37374375" x2="39.6048" y2="30.82625625" width="0.1524" layer="16"/>
-<wire x1="39.015528125" y1="25.784471875" x2="39.6048" y2="26.37374375" width="0.1524" layer="16"/>
-<wire x1="34.2567125" y1="32.48" x2="34" y2="32.48" width="0.1524" layer="16"/>
-<wire x1="34" y1="32.48" x2="32.385" y2="32.48" width="0.1524" layer="16"/>
-<wire x1="34.4053125" y1="32.6286" x2="34.2567125" y2="32.48" width="0.1524" layer="16"/>
-<wire x1="37.80245625" y1="32.6286" x2="34.4053125" y2="32.6286" width="0.1524" layer="16"/>
-<wire x1="39.6048" y1="30.82625625" x2="37.80245625" y2="32.6286" width="0.1524" layer="16"/>
-<wire x1="34.29" y1="35.56" x2="34" y2="32.48" width="0.1524" layer="16"/>
+<wire x1="39.6048" y1="30.82625625" x2="39.6048" y2="26.37374375" width="0.1524" layer="16"/>
+<wire x1="39" y1="25.76894375" x2="39.6048" y2="26.37374375" width="0.1524" layer="16"/>
 <wire x1="39" y1="23.24434375" x2="39" y2="23.7" width="0.1524" layer="1"/>
 <wire x1="39" y1="23.24434375" x2="38.8366" y2="23.08094375" width="0.1524" layer="1"/>
@@
 <wire x1="38.8366" y1="22.63905625" x2="39" y2="22.47565625" width="0.1524" layer="1"/>
 <wire x1="39" y1="22.47565625" x2="39" y2="22" width="0.1524" layer="1"/>
-<wire x1="39" y1="25.76894375" x2="39.015528125" y2="25.784471875" width="0.1524" layer="16"/>
 <wire x1="39" y1="22" x2="39" y2="22.47565625" width="0.1524" layer="16"/>
 <wire x1="39" y1="22.47565625" x2="38.8366" y2="22.63905625" width="0.1524" layer="16"/>
@@
 <wire x1="38.8366" y1="23.08094375" x2="39" y2="23.24434375" width="0.1524" layer="16"/>
 <wire x1="39" y1="23.24434375" x2="39" y2="25.76894375" width="0.1524" layer="16"/>
+<wire x1="32.385" y1="32.48" x2="32.925" y2="33.02" width="0.1524" layer="16"/>
+<wire x1="32.925" y1="33.02" x2="34.29" y2="33.02" width="0.1524" layer="16"/>
+<wire x1="34.29" y1="33.02" x2="37.41105625" y2="33.02" width="0.1524" layer="16"/>
+<wire x1="37.41105625" y1="33.02" x2="39.6048" y2="30.82625625" width="0.1524" layer="16"/>
+<wire x1="34.29" y1="35.56" x2="34.29" y2="33.02" width="0.1524" layer="16"/>
 </signal>
 <signal name="SWDIO">
@@
 <contactref element="U5" pad="SWDIO"/>
 <wire x1="35" y1="23.7" x2="35" y2="25" width="0.1524" layer="1"/>
-<wire x1="32.385" y1="33.75" x2="32.385" y2="35.615" width="0.1524" layer="16"/>
-<wire x1="32.385" y1="35.615" x2="31.75" y2="35.56" width="0.1524" layer="16"/>
 <wire x1="33.4" y1="26.6" x2="33.4" y2="33" width="0.1524" layer="1"/>
 <wire x1="33.4" y1="33" x2="32.65" y2="33.75" width="0.1524" layer="1"/>
 <wire x1="32.65" y1="33.75" x2="32.385" y2="33.75" width="0.1524" layer="1"/>
 <wire x1="35" y1="25" x2="33.4" y2="26.6" width="0.1524" layer="1"/>
+<wire x1="32.385" y1="33.75" x2="31.75" y2="34.385" width="0.1524" layer="16"/>
+<wire x1="31.75" y1="34.385" x2="31.75" y2="35.56" width="0.1524" layer="16"/>
 </signal>
 <signal name="UART-RX">
